Commit message: Use a deterministic map generation model for repeatability

File: gym_pybullet_drones/assets/cylinder.urdf (robot description, URDF)
Before this commit: robot cylinder, 1 links, 0 joints
Links:
- link base_link: geometry collision cylinder length=3 radius=0.25; visual cylinder length=3 radius=0.25
